File: Generator_ESP_board/Generator_ESP.kicad_pcb (KiCad board)
At the start: 2 copper layers, 67 parts, among them J1 Conn_01x02_Female, J10 Conn_01x03_Female, J11 Conn_01x02_Female, J2 Conn_01x02_Female, J3 Conn_01x04_Female, J4 Conn_01x02_Female, J5 Conn_02x08_Top_Bottom, J6 Conn_01x02_Female, J7 Conn_01x03_Female, J8 Conn_01x03_Female, J9 Conn_01x03_Female, K1 JOC-3FF, K2 JOC-3FF, Q1 2N2219, Q2 2N2219, Q3 BC847, Q4 BC847, SW1 SW_Push, SW2 SW_Push, U1 SFH617A-1, U2 SFH617A-1, U3 ESP8266_nodekit, U4 MAX483E, U5 MP1584EN

Commit message: adding latest pcb files
Parts:
- removed the R10 at (34.3, 72.1)
- removed the R12 at (86.4, 49.5)
- removed the R17 at (47.0, 81.5)
- removed the R2 at (89.9, 84.8)
- removed the R20 at (201.9, 36.6)
- removed R25: 24K, Resistor_SMD:R_0805_2012Metric_Pad1.20x1.40mm_HandSolder
- removed the R5 at (34.3, 77.5)
- removed the R8 at (30.5, 74.9)
- added H1: MountingHole, MountingHole:MountingHole_3.2mm_M3, F.Cu at (72.4, 131.6)
- added H2: MountingHole, MountingHole:MountingHole_3.2mm_M3, F.Cu at (72.4, 57.4)
- added H3: MountingHole, MountingHole:MountingHole_3.2mm_M3, F.Cu at (163.2, 57.4)
- added H4: MountingHole, MountingHole:MountingHole_3.2mm_M3, F.Cu at (163.3, 131.6)
- added R11: R_Small_US, Resistor_SMD:R_0805_2012Metric_Pad1.20x1.40mm_HandSolder, F.Cu at (156.0, 69.1)
- added R15: 62K, Resistor_SMD:R_0805_2012Metric_Pad1.20x1.40mm_HandSolder, F.Cu at (85.9, 87.4)
- added R18: 1K 0.25W, Resistor_SMD:R_0805_2012Metric_Pad1.20x1.40mm_HandSolder, F.Cu at (145.3, 90.8)
- added R22: 200K, Resistor_SMD:R_0805_2012Metric_Pad1.20x1.40mm_HandSolder, F.Cu at (88.4, 99.6)
- added R4: 20K, Resistor_SMD:R_0805_2012Metric_Pad1.20x1.40mm_HandSolder, F.Cu at (79.5, 97.3)
- added R7: 3.01K, Resistor_SMD:R_0805_2012Metric_Pad1.20x1.40mm_HandSolder, F.Cu at (75.7, 92.0)
- added R9: 0, Resistor_SMD:R_0805_2012Metric_Pad1.20x1.40mm_HandSolder, F.Cu at (79.5, 91.9)
- C1: footprint Capacitor_THT:C_Disc_D4.7mm_W2.5mm_P5.00mm -> Capacitor_SMD:C_0805_2012Metric
- C2: footprint Capacitor_SMD:C_1206_3216Metric -> Capacitor_SMD:C_2220_5650Metric
- C4: value 0.1uF -> CP1_Small
- C5: value CP1_Small -> 100n 50V Ceramic; footprint Capacitor_THT:C_Disc_D4.7mm_W2.5mm_P5.00mm -> Capacitor_SMD:C_0805_2012Metric
- C6: value 100n 50V Ceramic -> 2p 50V Ceramic
- C7: value 2p 50V Ceramic -> 820p 50V Ceramic
- C8: value 820p 50V Ceramic -> 100nF Ceramic
- D1, D2: footprint Diode_THT:D_DO-34_SOD68_P7.62mm_Horizontal -> Diode_SMD:D_MELF
- D5, D6: footprint Diode_THT:D_DO-34_SOD68_P7.62mm_Horizontal -> Diode_SMD:D_0805_2012Metric
- Q1, Q2: value 2N2219 -> Q_NPN_BEC
- Q3, Q4: value BC847 -> Q_NPN_BEC
- R16: value 62K -> 0
- R19: value 1K 0.25W -> SPARKFUN-RESISTORS_4.7KOHM-0603-1_10W-1%-Test
- R23: value 200K -> 100K
- R24: value 100K -> 24K
- moved D5 125.7 mm to (106.7, 117.1), turned to 90 degrees
- moved K1 117.6 mm to (111.3, 112.9), turned to 0 degrees
- moved J10 116.8 mm to (143.0, 128.8)
- moved K2 112.4 mm to (140.2, 112.0), turned to 0 degrees
- moved R17 111.8 mm to (106.7, 113.0)
- moved Q1 111.7 mm to (105.9, 109.0), turned to 90 degrees
- moved J9 109.2 mm to (126.7, 128.8)
- moved D6 102.8 mm to (156.4, 88.6)
- moved C8 99.8 mm to (140.3, 59.3), turned to 0 degrees
- moved R19 98.2 mm to (158.0, 56.5)
- moved Q2 93.6 mm to (151.0, 89.0), turned to 270 degrees
- moved R2 92.6 mm to (82.3, 67.1)
- moved D1 90.7 mm to (82.5, 75.0)
- moved R5 89.9 mm to (82.3, 69.1), turned to 180 degrees
- moved J3 86.3 mm to (116.5, 60.2)
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- renumbered R11 to R10, R13 to R12, R14 to R13, R15 to R14, R18 to R17, R3 to R2, R21 to R20, R22 to R21, R4 to R3, R6 to R5, R7 to R6, R9 to R8
Connections:
- C1 pad 1: +12V -> +5V
- C2 pad 1: +12V -> +5V
- C4 pad 1: GND -> Net-(C4-Pad1)
- C4 pad 2: +3V3 -> GND
- C5 pad 2: GND -> Net-(C5-Pad2)
- C6 pad 1: Net-(C6-Pad1) -> GND
- C8 pad 2: Net-(C8-Pad2) -> +5V
- D4 pad 1: Net-(C6-Pad2) -> Net-(C5-Pad2)
- J1 pad 1: 0 -> GND
- J2 pad 1: 0 -> GND
- J5 pad 10: GND -> /RST
- J5 pad 11: +3V3 -> /N6
- J5 pad 12: /N12 -> /N9
- J5 pad 13: /N13 -> /N7
- J5 pad 14: /Button1 -> GND
- J5 pad 15: /Button2 -> /N8
- J5 pad 2: /N2 -> +3V3
- J5 pad 3: /N3 -> /N2
- J5 pad 4: /N4 -> /Button2
- J5 pad 5: /N5 -> /N3
- J5 pad 6: /N6 -> /Button1
- J5 pad 7: /N7 -> /N4
- J5 pad 8: /N8 -> /EN
- J5 pad 9: /N9 -> /N5
- L1 pad 1: Net-(C6-Pad2) -> Net-(C5-Pad2)
- L1 pad 2: +12V -> +5V
- Q1 pad 1: GND -> Net-(Q1-Pad1)
- Q1 pad 2: Net-(Q1-Pad2) -> GND
- Q2 pad 1: GND -> Net-(Q2-Pad1)
- Q2 pad 2: Net-(Q2-Pad2) -> GND
- Q3 pad 1: GND -> Net-(Q3-Pad1)
- Q3 pad 2: Net-(Q3-Pad2) -> GND
- Q4 pad 1: GND -> Net-(Q4-Pad1)
- Q4 pad 2: Net-(Q4-Pad2) -> GND
- R1 pad 2: +12V -> +5V
- R10 pad 2: GND -> +3V3
- R12 pad 2: GND -> +3V3
- R13 pad 1: Net-(R14-Pad1) -> Net-(R13-Pad1)
- R14 pad 1: Net-(R14-Pad1) -> Net-(R13-Pad1)
- R16 pad 1: Net-(C7-Pad2) -> Net-(R16-Pad1)
- R16 pad 2: Net-(C8-Pad2) -> Net-(C5-Pad1)
- R17 pad 1: Net-(Q1-Pad2) -> Net-(Q1-Pad1)
- R17 pad 2: Net-(R18-Pad2) -> Net-(R17-Pad2)
- R19 pad 1: Net-(Q2-Pad2) -> Net-(J3-Pad3)
- R19 pad 2: Net-(R19-Pad2) -> Net-(J6-Pad1)
- R23 pad 1: GND -> Net-(C10-Pad2)
- R24 pad 1: Net-(C10-Pad2) -> GND
- R24 pad 2: Net-(R24-Pad2) -> Net-(R23-Pad2)
- R8 pad 1: Net-(R9-Pad1) (its old number) -> Net-(R8-Pad1)
- SW1 pad 2: +3V3 -> GND
- SW2 pad 2: +3V3 -> GND
- U3 pad 12: /N12 -> /EN
- U3 pad 13: +3V3 -> /RST
- U3 pad 22: Net-(Q3-Pad2) -> Net-(Q3-Pad1)
- U3 pad 23: Net-(Q4-Pad2) -> Net-(Q4-Pad1)
- U4 pad 2: Net-(U4-Pad2) -> /N1
- U4 pad 3: Net-(U4-Pad2) -> /N1
- U5 pad 1: Net-(C6-Pad2) -> Net-(C5-Pad2)
- U5 pad 2: Net-(R24-Pad2) -> Net-(R23-Pad2)
- U5 pad 3: Net-(C7-Pad2) -> Net-(C6-Pad2)
- U5 pad 6: Net-(R23-Pad2) -> Net-(R22-Pad2)
- U5 pad 8: Net-(R17-Pad1) -> Net-(R16-Pad1)
Routing:
- net +5V: track 0.00 -> 278.4 mm, vias 0 -> 5
- net /Button1: track 0.00 -> 150.3 mm, vias 0 -> 3
- net +3V3: track 0.00 -> 147.6 mm, vias 0 -> 3
- net /N1: track 0.00 -> 111.8 mm, vias 0 -> 5
- net /Button2: track 0.00 -> 106.3 mm, vias 0 -> 3
- net Net-(U3-Pad19): track 0.00 -> 100.3 mm, vias 0 -> 6
- net Net-(C10-Pad2): track 0.00 -> 90.6 mm, vias 0 -> 2
- net Net-(R13-Pad1): track 0.00 -> 65.2 mm, vias 0 -> 2
- net /N3: track 0.00 -> 63.8 mm
- net Net-(U3-Pad18): track 0.00 -> 63.6 mm, vias 0 -> 2
- net /N9: track 0.00 -> 62.8 mm
- net /RST: track 0.00 -> 62.4 mm, vias 0 -> 2
- net /N4: track 0.00 -> 61.3 mm
- net /N5: track 0.00 -> 58.8 mm
- net /N6: track 0.00 -> 56.9 mm
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- added copper zone on B.Cu, net GND
Other:
- board outline added: 99.1 x 82.3 mm
- net class 12V added: clearance 0.2, trace_width 1.36, via_dia 1.91, via_drill 0.95
- net class 5V added: clearance 0.2, trace_width 0.7, via_dia 1.25, via_drill 0.625
- net class GND added: clearance 0.2, trace_width 0.7, via_dia 1.25, via_drill 0.625
- net class Relay_10A added: clearance 0.8, trace_width 3, via_dia 3.55, via_drill 1.75
- board text added: "5V"
- board text added: "Config"
- board text added: "GND"
- board text added: "Giga Technology"
- board text added: "Relay Out"
- board text added: "SN: _______________"
- board text added: "Servo Out"
- board text added: "Start/Stop"
- board text added: "Ver. 1.0"
