File: Generator_ESP_board/Generator_ESP.sch (KiCad schematic (older format))
At the start: 68 parts, among them J1 Conn_01x02_Female, J10 Conn_01x03_Female, J11 Conn_01x02_Female, J2 Conn_01x02_Female, J3 Conn_01x04_Female, J4 Conn_01x02_Female, J5 Conn_02x08_Top_Bottom, J6 Conn_01x02_Female, J7 Conn_01x03_Female, J8 Conn_01x03_Female, J9 Conn_01x03_Female, K1 JOC-3FF, K2 JOC-3FF, Q1 2N2219, Q2 2N2219, Q3 BC847, Q4 BC847, SW1 SW_Push, SW2 SW_Push, U1 SFH617A-1, U2 SFH617A-1, U3 ESP8266_nodekit, U4 MAX483E, U5 MP1584EN

Commit message: adding latest pcb files
Parts:
- removed C4: 0.1uF, Capacitor_SMD:C_0805_2012Metric, symbol Device:C_Small
- removed Q1, Q2: 2N2219, Package_TO_SOT_SMD:SOT-23, symbol Transistor_BJT:2N2219
- removed Q3, Q4: BC847, Package_TO_SOT_SMD:SOT-23, symbol Transistor_BJT:2N2219
- removed R2, R5: 1K, Resistor_SMD:R_0805_2012Metric_Pad1.20x1.40mm_HandSolder, symbol Generator_ESP-rescue:SPARKFUN-RESISTORS_4.7KOHM-0603-1_10W-1%-Test
- added C8: 100nF Ceramic, Capacitor_SMD:C_0805_2012Metric, symbol Device:C_Small
- added H1, H2, H3, H4: MountingHole, MountingHole:MountingHole_3.2mm_M3, symbol Mechanical:MountingHole
- added Q1, Q2, Q3, Q4: Q_NPN_BEC, Package_TO_SOT_SMD:SOT-23, symbol Device:Q_NPN_BEC
- C1: footprint Capacitor_THT:C_Disc_D4.7mm_W2.5mm_P5.00mm -> Capacitor_SMD:C_0805_2012Metric
- C2: footprint Capacitor_SMD:C_1206_3216Metric -> Capacitor_SMD:C_2220_5650Metric
- C4: renamed from C5; footprint Capacitor_THT:C_Disc_D4.7mm_W2.5mm_P5.00mm -> Capacitor_SMD:C_0805_2012Metric
- D1, D2: footprint Diode_THT:D_DO-34_SOD68_P7.62mm_Horizontal -> Diode_SMD:D_MELF
- D5, D6: footprint Diode_THT:D_DO-34_SOD68_P7.62mm_Horizontal -> Diode_SMD:D_0805_2012Metric
- renumbered C6 to C5, C7 to C6, C8 to C7, R12 to R10, R13 to R11, R14 to R12, R15 to R13, R16 to R14, R17 to R15, R18 to R16, R19 to R17, R20 to R18, R21 to R19, R3 to R2, R22 to R20, R23 to R21, R24 to R22, R25 to R23, R26 to R24, R4 to R3, R6 to R4, R7 to R5, R8 to R6, R9 to R7, R10 to R8, R11 to R9
Connections:
- net 0 is gone; now on net GND: J1.1 (Pin_1), J2.1 (Pin_1)
- net +12V: no longer C1.1, C2.1, L1.2, R1.2, R4.2
- net +3V3: now also J5.2 (Pin_2), R10.2, R12.2; no longer J5.11 (Pin_11), SW1.2, SW2.2
- net +5V: now also C1.1, C2.1, L1.2, R1.2, R4.2, C8.2
- net Button1: now also J5.6 (Pin_6); no longer J5.14 (Pin_14)
- net Button2: now also J5.4 (Pin_4); no longer J5.15 (Pin_15)
- net EN: now also J5.8 (Pin_8)
- net GND: now also J5.14 (Pin_14), SW1.2, SW2.2, C8.1, Q1.2 (E), Q2.2 (E), Q3.2 (E), Q4.2 (E); no longer J5.10 (Pin_10), R10.2, R12.2
- net N1: now also U4.2 (~RE), U4.3 (DE)
- net N2: now also J5.3 (Pin_3); no longer J5.2 (Pin_2)
- net N3: now also J5.5 (Pin_5); no longer J5.3 (Pin_3)
- net N4: now also J5.7 (Pin_7); no longer J5.4 (Pin_4)
- net N5: now also J5.9 (Pin_9); no longer J5.5 (Pin_5)
- net N6: now also J5.11 (Pin_11); no longer J5.6 (Pin_6)
- net N7: now also J5.13 (Pin_13); no longer J5.7 (Pin_7)
- net N8: now also J5.15 (Pin_15); no longer J5.8 (Pin_8)
- net N9: now also J5.12 (Pin_12); no longer J5.9 (Pin_9)
- net RST: now also J5.10 (Pin_10)
- net at D6.2 (A), K2.2: now also Q2.3 (C)
- net at D5.2 (A), K1.2: now also Q1.3 (C)
- net at R17.1: now also Q1.1 (B)
- net at R18.1: now also Q2.1 (B)
- net at U3.22 (D6): now also Q3.1 (B)
- net at J7.1 (Pin_1), R20.1: now also Q3.3 (C)
- net at U3.23 (D5): now also Q4.1 (B)
- net at J8.1 (Pin_1), R21.1: now also Q4.3 (C)
